File: PCB_files/PD240W_kicad.kicad_pcb (KiCad board)
At the start: 6 copper layers, 66 x 66 mm, 299 parts, among them J1 DX07S024JJ2R1300, J2 61300411121, J3 24.245.1, J4 24.245.2, J5 1935776, J6 1935776, J7 61300411121, J8 AFC07-S12FCA-00, Q1 AGM612AP, Q2 AO3404A, Q3 SQJB90EP-T1_GE3, Q4 AO3404A, Q5 AO3404A, Q6 AO3404A, Q7 AO3404A, U1 TPD4S480RUKR, U10 W25Q128JVPIQ, U11 LMR16006XDDCR, U12 LMR16006XDDCR, U2 LM2765, U3 TPS26750SRSMR, U4 LTC7004x, U5 74LVC1G08SE-7, U6 CAT24C512YI-GT3, U7 SN74LVC1G17DBVR, U8 INA228AIDGSR, U9 RP2040, Y1 ABM8-272-T3

Commit message: Update 17V output to 5V output
Parts:
- removed L2: 68uH 0.55A 0.91Ohm, Altium_port:SWPA4030S220MT
- removed R86: 10k 1%, Altium_port:resc_1005_04_n
- removed R89, R90: 4.7k 1%, Altium_port:resc_1005_04_m
- added L3: 33uH 1.3A 244mOhm, Inductor_SMD:L_APV_ANR5020, F.Cu at (161.2, 72.9)
- added R91: 10k 1%, Altium_port:resc_1005_04_n, F.Cu at (159.1, 79.9)
- added R92: 10k 1%, Altium_port:resc_1005_04_n, F.Cu at (159.1, 79.0)
- added R93: 10k 1%, Altium_port:resc_1005_04_n, F.Cu at (159.1, 78.1)
- C67: value 10u X7R 63V -> 22u X7R 25V
- R88: value 100k 1% -> 1k 1%
- moved R88 9.74 mm to (169.7, 75.3), turned to -90 degrees
- moved R59 2.46 mm to (161.8, 81.0)
- moved TP66 2.20 mm to (162.4, 79.9)
- moved TP64 1.70 mm to (163.8, 69.9)
- moved FD2 1.60 mm to (159.4, 66.9)
- moved C63 0.82 mm to (158.8, 76.4), turned to 180 degrees
- moved R87 0.50 mm to (159.1, 81.0)
- moved TP35 0.40 mm to (164.1, 64.2)
Connections:
- net /Project Architecture/MCU - Unit/17V_EN_R renamed /Project Architecture/MCU - Unit/5V_EN_R
- net /Project Architecture/Power - Generation/17V_CB renamed /Project Architecture/Power - Generation/5V_CB
- net /Project Architecture/Power - Generation/17V_SW renamed /Project Architecture/Power - Generation/5V_SW
- C67 pad 1: +17V -> +5V
- D14 pad 2: /Project Architecture/Power - Generation/LED_17V_A -> /Project Architecture/Power - Generation/LED_5V_A
- F2 pad 1: +17V -> +5V
- F2 pad 2: /Project Architecture/Power - Output/17V_FUSED -> /Project Architecture/Power - Output/5V_FUSED
- J6 pad 1: /Project Architecture/Power - Output/17V_FUSED -> /Project Architecture/Power - Output/5V_FUSED
- J6 pad 2: /Project Architecture/Power - Output/17V_FUSED -> GND
- R59 pad 2: /Project Architecture/MCU - Unit/17V_EN -> /Project Architecture/MCU - Unit/5V_EN
- R85 pad 1: /Project Architecture/MCU - Unit/17V_EN -> /Project Architecture/Power - Generation/5V_EN
- R87 pad 1: +17V -> +5V
- R88 pad 1: Net-(R87-Pad2) -> +5V
- R88 pad 2: /Project Architecture/Power - Generation/17V_FB -> /Project Architecture/Power - Generation/LED_5V_A
- TP64 pad 1: +17V -> +5V
- TP66 pad 1: /Project Architecture/MCU - Unit/17V_EN -> /Project Architecture/Power - Generation/5V_EN
- U12 pad 3: /Project Architecture/Power - Generation/17V_FB -> /Project Architecture/Power - Generation/5V_FB
- U12 pad 4: /Project Architecture/MCU - Unit/17V_EN -> /Project Architecture/Power - Generation/5V_EN
Routing:
- net +5V: track 0.00 -> 27.1 mm, vias 0 -> 2
- net +17V: track 25.8 -> 0.00 mm, vias 2 -> 0
- net /Project Architecture/MCU - Unit/17V_EN: track 6.84 -> 0.00 mm
- net /Project Architecture/Power - Generation/LED_5V_A: track 0.00 -> 6.18 mm
- net /Project Architecture/Power - Generation/LED_17V_A: track 6.12 -> 0.00 mm
- net /Project Architecture/Power - Generation/5V_SW: track 0.00 -> 4.16 mm
- net (no net): track 0.00 -> 3.71 mm
- net /Project Architecture/MCU - Unit/5V_EN_R: track 12.2 -> 15.5 mm
- net /Project Architecture/Power - Generation/17V_FB: track 2.74 -> 0.00 mm
- net /Project Architecture/MCU - Unit/SWDIO_R: track 30.5 -> 33.0 mm
- net /Project Architecture/Power - Generation/5V_FB: track 0.00 -> 2.33 mm
- net /Project Architecture/MCU - Unit/SWCLK_R: track 29.0 -> 31.0 mm
- net Net-(R89-Pad2): track 1.30 -> 0.00 mm
- net Net-(R92-Pad2): track 0.00 -> 0.90 mm
- net /Project Architecture/Power - Generation/5V_CB: track 1.87 -> 1.36 mm
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- added copper zone on F.Cu, net +5V
- added copper zone on F.Cu, net /Project Architecture/Power - Output/5V_FUSED
- removed copper zone on F.Cu, net +17V
- removed copper zone on F.Cu, net /Project Architecture/Power - Output/17V_FUSED
Other:
- board text removed: "17"
- board text removed: "Heng"
- board text removed: "Théo"
