File: PCB_files/PD240W_kicad.kicad_pcb (KiCad board)
At the start: 6 copper layers, 66 x 66 mm, 299 parts, among them J1 DX07S024JJ2R1300, J2 61300411121, J3 24.245.1, J4 24.245.2, J5 1935776, J6 1935776, J7 61300411121, J8 AFC07-S12FCA-00, Q1 AGM612AP, Q2 AO3404A, Q3 SQJB90EP-T1_GE3, Q4 AO3404A, Q5 AO3404A, Q6 AO3404A, Q7 AO3404A, U1 TPD4S480RUKR, U10 W25Q128JVPIQ, U11 LMR16006XDDCR, U12 LMR16006XDDCR, U2 LM2765, U3 TPS26750SRSMR, U4 LTC7004x, U5 74LVC1G08SE-7, U6 CAT24C512YI-GT3, U7 SN74LVC1G17DBVR, U8 INA228AIDGSR, U9 RP2040, Y1 ABM8-272-T3

Commit message: Fix production files
Parts:
- renumbered C17 to C10, C19 to C11, C10 to C12, C20 to C13, C11 to C14, C12 to C15, C22 to C16, C13 to C17, C15 to C18, C14 to C19, C7 to C2, C16 to C20, C18 to C22, C26 to C23, C27 to C24, C23 to C25, C24 to C26, C25 to C27, C2 to C3, C44 to C31, C45 to C32, C46 to C33, C31 to C34, C33 to C35, C32 to C37, C34 to C38, C37 to C39, C8 to C4, C35 to C40, C38 to C41, C39 to C42, C40 to C43, C41 to C44, C42 to C45, C43 to C46, C53 to C47, C49 to C48, C50 to C49, C3 to C5, C54 to C50, C48 to C51, C47 to C52, C51 to C53, C52 to C54, C64 to C55, C65 to C57, C57 to C58, C66 to C59, C4 to C6, C58 to C60, C62 to C61, C63 to C62, C55 to C63, C67 to C64, C59 to C65, C60 to C66, C61 to C67, C5 to C7, C6 to C8, D9 to D10, D13 to D12, D12 to D13, D7 to D5, D5 to D6, D6 to D7, D10 to D9, J6 to J5, J5 to J6, JP2 to JP1, JP3 to JP10, JP1 to JP2, JP5 to JP3, JP7 to JP4, JP4 to JP5, JP8 to JP7, JP9 to JP8, JP10 to JP9, L3 to L1, L1 to L2, MH2 to MH1, MH4 to MH2, MH5 to MH4, MH1 to MH5, Q4 to Q3, Q5 to Q4, Q3 to Q5, R2 to R1, R11 to R10, R12 to R11, R13 to R12, R21 to R13, R15 to R14, R16 to R15, R19 to R16, R18 to R17, R7 to R18, R14 to R19, R6 to R2, R17 to R20, R20 to R21, R27 to R22, R29 to R23, R31 to R24, R28 to R25, R30 to R26, R32 to R27, R23 to R28, R22 to R29, R1 to R3, R24 to R30, R26 to R31, R25 to R32, R41 to R35, R63 to R36, R64 to R37, R66 to R38, R40 to R39, R3 to R4, R42 to R40, R43 to R41, R44 to R42, R45 to R43, R46 to R44, R38 to R45, R39 to R46, R35 to R47, R47 to R48, R48 to R49, R4 to R5, R49 to R50, R5 to R6, R65 to R62, R62 to R63, R67 to R64, R37 to R65, R36 to R66, R50 to R67, R78 to R68, R76 to R69, R8 to R7, R69 to R70, R68 to R71, R70 to R72, R71 to R73, R72 to R74, R79 to R75, R77 to R76, R74 to R77, R75 to R78, R73 to R79, R9 to R8, R85 to R80, R84 to R83, R87 to R84, R91 to R85, R92 to R86, R93 to R87, R80 to R88, R83 to R89, R10 to R9, R88 to R90, S4 to S3, S3 to S4, TP3 to TP1, TP1 to TP10, TP2 to TP11, TP4 to TP12, TP6 to TP13, TP17 to TP15, TP19 to TP16, TP21 to TP17, TP23 to TP18, TP25 to TP19, TP5 to TP2, TP15 to TP20, TP18 to TP21, TP20 to TP22, TP22 to TP23, TP26 to TP25, TP16 to TP26, TP7 to TP3, TP47 to TP33, TP48 to TP34, TP49 to TP35, TP50 to TP36, TP33 to TP37, TP34 to TP38, TP35 to TP39, TP8 to TP4, TP36 to TP40, TP37 to TP41, TP38 to TP42, TP39 to TP43, TP40 to TP44, TP41 to TP45, TP42 to TP46, TP43 to TP47, TP44 to TP48, TP45 to TP49, TP9 to TP5, TP46 to TP50, TP53 to TP52, TP52 to TP53, TP10 to TP6, TP11 to TP7, TP12 to TP8, TP13 to TP9, U9 to U10, U12 to U11, U11 to U12, U3 to U2, U6 to U3, U2 to U4, U4 to U6, U8 to U7, U7 to U8, U10 to U9
Connections:
- R80 pad 1: /Project Architecture/Power - Generation/5V_EN -> /Project Architecture/MCU - Unit/5V_EN
- TP66 pad 1: /Project Architecture/Power - Generation/5V_EN -> /Project Architecture/MCU - Unit/5V_EN
- U11 pad 4: /Project Architecture/Power - Generation/5V_EN -> /Project Architecture/MCU - Unit/5V_EN
Routing:
- net /Project Architecture/MCU - Unit/5V_EN: track 0.00 -> 3.71 mm
- net (no net): track 3.71 -> 0.00 mm
Other:
- board text added: "8/15/2026"
- board text added: "Rev v1.1"
- board text removed: "12/25"
