File: PCB_files/power_output.kicad_sch (KiCad schematic)
At the start: 14 parts, among them J3 24.245.1, J4 24.245.2, J5 1935776, J6 1935776

Commit message: Update 17V output to 5V output
Connections:
- net GND: now also J6.2 (Pin_2)
- net +17V renamed +5V
- net 17V_FUSED renamed 5V_FUSED
- net 5V_FUSED: no longer J6.2 (Pin_2)
Other:
- note added: "Screw Terminals for 5V"
- note removed: "Screw Terminals for 17V"
