File: PCB_files/power_output.kicad_sch (KiCad schematic)
At the start: 14 parts, among them J3 24.245.1, J4 24.245.2, J5 1935776, J6 1935776

Commit message: Fix production files
Parts:
- C28, C29: MFR Part # (none) -> GRM32ER71J106KA12L; Manufacturer Part Number GRM32ER71J106KA12L -> (none)
- C30: MFR Part # (none) -> CL10B104KC8NNNC; Manufacturer Part Number CL10B104KC8NNNC -> (none)
- D8: MFR Part # (none) -> SMAJ48A; Manufacturer Part Number SMAJ48A -> (none)
- F1, F2: MFR Part # (none) -> FSMD020-1206-R; Manufacturer Part Number FSMD020-1206-R -> (none)
- J3: MFR Part # (none) -> 24.245.1; Manufacturer Part Number 24.245.1 -> (none)
- J4: MFR Part # (none) -> 24.245.2; Manufacturer Part Number 24.245.2 -> (none)
- J5: renamed from J6; MFR Part # (none) -> 1935776; Manufacturer Part Number 1935776 -> (none)
- J6: renamed from J5; MFR Part # (none) -> 1935776; Manufacturer Part Number 1935776 -> (none)
- R33, R34: MFR Part # (none) -> RC0402FR-0733KL; Manufacturer Part Number RC0402FR-0733KL -> (none)
- TP31, TP32: MFR Part # (none) -> 5001; Manufacturer Part Number 5001 -> (none)
Changed lines of the file:
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@@
 	(title_block
 		(title "Power - Output")
-		(date "2026-02-27")
+		(date "2026-08-15")
 		(rev "${REVISION}")
 	)
@@
 		(dnp no)
 		(fields_autoplaced yes)
-		(property "Reference" "#PWR0183"
+		(property "Reference" "#PWR0112"
 			(at 238.76 214.63 0)
 			(hide yes)
@@
 			(project "PD240W_kicad"
 				(path "/f9e05184-c88b-4a88-ae9c-ab2bdb32be7c/c5103ceb-5325-4a84-a025-9638a412984e/dead5858-73e4-406c-878c-50ea6c895061"
-					(reference "#PWR0183")
+					(reference "#PWR0112")
 					(unit 1)
 				)
@@
 		(dnp no)
 		(fields_autoplaced yes)
-		(property "Reference" "#PWR0180"
+		(property "Reference" "#PWR0107"
 			(at 109.22 76.2 0)
 			(hide yes)
@@
 			(project "PD240W_kicad"
 				(path "/f9e05184-c88b-4a88-ae9c-ab2bdb32be7c/c5103ceb-5325-4a84-a025-9638a412984e/dead5858-73e4-406c-878c-50ea6c895061"
-					(reference "#PWR0180")
+					(reference "#PWR0107")
 					(unit 1)
 				)
@@
 			)
 		)
-		(property "Manufacturer Part Number" "SMAJ48A"
+		(property "MFR Part #" "SMAJ48A"
 			(at 250.19 104.14 90)
 			(hide yes)
@@
 			)
 		)
-		(property "Manufacturer Part Number" "24.245.2"
+		(property "MFR Part #" "24.245.2"
 			(at 275.59 123.19 0)
 			(hide yes)
@@
 		(in_pos_files yes)
 		(dnp no)
-		(property "Reference" "#PWR0114"
+		(property "Reference" "#PWR0110"
 			(at 238.76 186.69 0)
 			(hide yes)
@@
 			(project "PD240W_kicad"
 				(path "/f9e05184-c88b-4a88-ae9c-ab2bdb32be7c/c5103ceb-5325-4a84-a025-9638a412984e/dead5858-73e4-406c-878c-50ea6c895061"
-					(reference "#PWR0114")
+					(reference "#PWR0110")
 					(unit 1)
 				)
@@
 			)
 		)
-		(property "Manufacturer Part Number" "24.245.1"
+		(property "MFR Part #" "24.245.1"
 			(at 275.59 68.58 0)
 			(hide yes)
@@
 		(in_pos_files yes)
 		(dnp no)
-		(property "Reference" "J5"
+		(property "Reference" "J6"
 			(at 285.75 189.23 0)
 			(show_name no)
@@
 			)
 		)
-		(property "Manufacturer Part Number" "1935776"
+		(property "MFR Part #" "1935776"
 			(at 283.21 189.23 0)
 			(hide yes)
@@
 			(project "PD240W_kicad"
 				(path "/f9e05184-c88b-4a88-ae9c-ab2bdb32be7c/c5103ceb-5325-4a84-a025-9638a412984e/dead5858-73e4-406c-878c-50ea6c895061"
-					(reference "J5")
+					(reference "J6")
 					(unit 1)
 				)
@@
 			)
 		)
-		(property "Manufacturer Part Number" "FSMD020-1206-R"
+		(property "MFR Part #" "FSMD020-1206-R"
 			(at 256.54 210.82 90)
 			(hide yes)
@@
 			)
 		)
-		(property "Manufacturer Part Number" "5001"
+		(property "MFR Part #" "5001"
 			(at 245.19 76.2 0)
 			(hide yes)
@@
 			)
 		)
-		(property "Manufacturer Part Number" "FSMD020-1206-R"
+		(property "MFR Part #" "FSMD020-1206-R"
 			(at 256.54 186.69 90)
 			(hide yes)
@@
 		(in_pos_files yes)
 		(dnp no)
-		(property "Reference" "#PWR0111"
+		(property "Reference" "#PWR0116"
 			(at 300.99 83.82 0)
 			(hide yes)
@@
 			(project "PD240W_kicad"
 				(path "/f9e05184-c88b-4a88-ae9c-ab2bdb32be7c/c5103ceb-5325-4a84-a025-9638a412984e/dead5858-73e4-406c-878c-50ea6c895061"
-					(reference "#PWR0111")
+					(reference "#PWR0116")
 					(unit 1)
 				)
@@
 			)
 		)
-		(property "Manufacturer Part Number" "GRM32ER71J106KA12L"
+		(property "MFR Part #" "GRM32ER71J106KA12L"
 			(at 180.34 104.14 0)
 			(hide yes)
@@
 		(in_pos_files yes)
 		(dnp no)
-		(property "Reference" "#PWR0178"
+		(property "Reference" "#PWR0113"
 			(at 238.76 218.44 0)
 			(hide yes)
@@
 			(project "PD240W_kicad"
 				(path "/f9e05184-c88b-4a88-ae9c-ab2bdb32be7c/c5103ceb-5325-4a84-a025-9638a412984e/dead5858-73e4-406c-878c-50ea6c895061"
-					(reference "#PWR0178")
+					(reference "#PWR0113")
 					(unit 1)
 				)
@@
 			)
 		)
-		(property "Manufacturer Part Number" "RC0402FR-0733KL"
+		(property "MFR Part #" "RC0402FR-0733KL"
 			(at 236.22 115.57 0)
 			(hide yes)
@@
 			)
 		)
-		(property "Manufacturer Part Number" "5001"
+		(property "MFR Part #" "5001"
 			(at 255.19 130.81 0)
 			(hide yes)
@@
 		(in_pos_files yes)
 		(dnp no)
-		(property "Reference" "#PWR0112"
+		(property "Reference" "#PWR0115"
 			(at 273.05 138.43 0)
 			(hide yes)
@@
 			(project "PD240W_kicad"
 				(path "/f9e05184-c88b-4a88-ae9c-ab2bdb32be7c/c5103ceb-5325-4a84-a025-9638a412984e/dead5858-73e4-406c-878c-50ea6c895061"
-					(reference "#PWR0112")
+					(reference "#PWR0115")
 					(unit 1)
 				)
@@
 		(in_pos_files yes)
 		(dnp no)
-		(property "Reference" "J6"
+		(property "Reference" "J5"
 			(at 284.48 210.82 0)
 			(show_name no)
@@
 			)
 		)
-		(property "Manufacturer Part Number" "1935776"
+		(property "MFR Part #" "1935776"
 			(at 281.94 210.82 0)
 			(hide yes)
@@
 			(project "PD240W_kicad"
 				(path "/f9e05184-c88b-4a88-ae9c-ab2bdb32be7c/c5103ceb-5325-4a84-a025-9638a412984e/dead5858-73e4-406c-878c-50ea6c895061"
-					(reference "J6")
+					(reference "J5")
 					(unit 1)
 				)
@@
 			)
 		)
-		(property "Manufacturer Part Number" "RC0402FR-0733KL"
+		(property "MFR Part #" "RC0402FR-0733KL"
 			(at 236.22 86.36 0)
 			(hide yes)
@@
 		(in_pos_files yes)
 		(dnp no)
-		(property "Reference" "#PWR0115"
+		(property "Reference" "#PWR0111"
 			(at 238.76 194.31 0)
 			(hide yes)
@@
 			(project "PD240W_kicad"
 				(path "/f9e05184-c88b-4a88-ae9c-ab2bdb32be7c/c5103ceb-5325-4a84-a025-9638a412984e/dead5858-73e4-406c-878c-50ea6c895061"
-					(reference "#PWR0115")
+					(reference "#PWR0111")
 					(unit 1)
 				)
@@
 		(in_pos_files yes)
 		(dnp no)
-		(property "Reference" "#PWR0108"
+		(property "Reference" "#PWR0109"
 			(at 180.34 76.2 0)
 			(hide yes)
@@
 			(project "PD240W_kicad"
 				(path "/f9e05184-c88b-4a88-ae9c-ab2bdb32be7c/c5103ceb-5325-4a84-a025-9638a412984e/dead5858-73e4-406c-878c-50ea6c895061"
-					(reference "#PWR0108")
+					(reference "#PWR0109")
 					(unit 1)
 				)
@@
 			)
 		)
-		(property "Manufacturer Part Number" "CL10B104KC8NNNC"
+		(property "MFR Part #" "CL10B104KC8NNNC"
 			(at 215.9 104.14 0)
 			(hide yes)
@@
 		(in_pos_files yes)
 		(dnp no)
-		(property "Reference" "#PWR0109"
+		(property "Reference" "#PWR0108"
 			(at 113.03 83.82 0)
 			(hide yes)
@@
 			(project "PD240W_kicad"
 				(path "/f9e05184-c88b-4a88-ae9c-ab2bdb32be7c/c5103ceb-5325-4a84-a025-9638a412984e/dead5858-73e4-406c-878c-50ea6c895061"
-					(reference "#PWR0109")
+					(reference "#PWR0108")
 					(unit 1)
 				)
@@
 		(in_pos_files yes)
 		(dnp no)
-		(property "Reference" "#PWR0113"
+		(property "Reference" "#PWR0117"
 			(at 300.99 138.43 0)
 			(hide yes)
@@
 			(project "PD240W_kicad"
 				(path "/f9e05184-c88b-4a88-ae9c-ab2bdb32be7c/c5103ceb-5325-4a84-a025-9638a412984e/dead5858-73e4-406c-878c-50ea6c895061"
-					(reference "#PWR0113")
+					(reference "#PWR0117")
 					(unit 1)
 				)
@@
 			)
 		)
-		(property "Manufacturer Part Number" "GRM32ER71J106KA12L"
+		(property "MFR Part #" "GRM32ER71J106KA12L"
 			(at 198.12 104.14 0)
 			(hide yes)
@@
 		(in_pos_files yes)
 		(dnp no)
-		(property "Reference" "#PWR0110"
+		(property "Reference" "#PWR0114"
 			(at 273.05 83.82 0)
 			(hide yes)
@@
 			(project "PD240W_kicad"
 				(path "/f9e05184-c88b-4a88-ae9c-ab2bdb32be7c/c5103ceb-5325-4a84-a025-9638a412984e/dead5858-73e4-406c-878c-50ea6c895061"
-					(reference "#PWR0110")
+					(reference "#PWR0114")
 					(unit 1)
 				)
