File: PCB_files/Block Diagram.kicad_sch (KiCad schematic)
At the start: 0 parts

Commit message: Fix production files
Other:
- title: Block Diagram -> Power - Output
Changed lines of the file:
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@@
 	(paper "A3")
 	(title_block
-		(title "Block Diagram")
+		(title "Power - Output")
 		(date "2026-02-27")
 		(rev "${REVISION}")
