File: PCB_files/user_interface.kicad_sch (KiCad schematic)
At the start: 41 parts, among them J8 AFC07-S12FCA-00, Q7 AO3404A

Commit message: Fix production files
Parts:
- C47: renamed from C53; MFR Part # (none) -> CL10B104KC8NNNC; Manufacturer Part Number CL10B104KC8NNNC -> (none)
- C48: renamed from C49; MFR Part # (none) -> CL10B104KC8NNNC; Manufacturer Part Number CL10B104KC8NNNC -> (none)
- C49: renamed from C50; MFR Part # (none) -> CL10B104KC8NNNC; Manufacturer Part Number CL10B104KC8NNNC -> (none)
- C50: renamed from C54; MFR Part # (none) -> CL10B104KC8NNNC; Manufacturer Part Number CL10B104KC8NNNC -> (none)
- C51: renamed from C48; MFR Part # (none) -> CL10B104KC8NNNC; Manufacturer Part Number CL10B104KC8NNNC -> (none)
- C52: renamed from C47; MFR Part # (none) -> CL10B104KC8NNNC; Manufacturer Part Number CL10B104KC8NNNC -> (none)
- C53: renamed from C51; MFR Part # (none) -> CC0805KKX7R0BB105; Manufacturer Part Number CC0805KKX7R0BB105 -> (none)
- C54: renamed from C52; MFR Part # (none) -> CL10B104KC8NNNC; Manufacturer Part Number CL10B104KC8NNNC -> (none)
- D11: MFR Part # (none) -> SK6812-EC20; Manufacturer Part Number SK6812-EC20 -> (none)
- DSP1: MFR Part # (none) -> HS20HS072RX; Manufacturer Part Number HS20HS072RX -> (none)
- J8: MFR Part # (none) -> AFC07-S12FCA-00; Manufacturer Part Number AFC07-S12FCA-00 -> (none)
- PZ1: MFR Part # (none) -> FUET-9018; Manufacturer Part Number FUET-9018 -> (none)
- Q7: MFR Part # (none) -> AO3404A; Manufacturer Part Number AO3404A -> (none)
- R68: renamed from R78; MFR Part # (none) -> RC0402FR-0733KL; Manufacturer Part Number RC0402FR-0733KL -> (none)
- R69: renamed from R76; MFR Part # (none) -> 0402WGF1002TCE; Manufacturer Part Number 0402WGF1002TCE -> (none)
- R70: renamed from R69; MFR Part # (none) -> 0402WGF1002TCE; Manufacturer Part Number 0402WGF1002TCE -> (none)
- R71: renamed from R68; MFR Part # (none) -> 0402WGF3300TCE; Manufacturer Part Number 0402WGF3300TCE -> (none)
- R72: renamed from R70; MFR Part # (none) -> 0402WGF1002TCE; Manufacturer Part Number 0402WGF1002TCE -> (none)
- R73: renamed from R71; MFR Part # (none) -> 0402WGF1002TCE; Manufacturer Part Number 0402WGF1002TCE -> (none)
- R74: renamed from R72; MFR Part # (none) -> RC0402FR-0733KL; Manufacturer Part Number RC0402FR-0733KL -> (none)
- R75: renamed from R79; MFR Part # (none) -> RC0402FR-0733KL; Manufacturer Part Number RC0402FR-0733KL -> (none)
- R76: renamed from R77; MFR Part # (none) -> 0402WGF1002TCE; Manufacturer Part Number 0402WGF1002TCE -> (none)
- R77: renamed from R74; MFR Part # (none) -> RC0402FR-0727RL; Manufacturer Part Number RC0402FR-0727RL -> (none)
- R78: renamed from R75; MFR Part # (none) -> 0402WGF1003TCE; Manufacturer Part Number 0402WGF1003TCE -> (none)
- R79: renamed from R73; MFR Part # (none) -> FRC0402F3R90TS; Manufacturer Part Number FRC0402F3R90TS -> (none)
- S3: renamed from S4; MFR Part # (none) -> GT-TC120A-H120-L1; Manufacturer Part Number GT-TC120A-H120-L1 -> (none)
- S4: renamed from S3; MFR Part # (none) -> PEC11R-4215F-S0024; Manufacturer Part Number PEC11R-4215F-S0024 -> (none)
- S5: MFR Part # (none) -> GT-TC120A-H120-L1; Manufacturer Part Number GT-TC120A-H120-L1 -> (none)
- renumbered TP53 to TP52, TP52 to TP53
Other:
- title: User - Interface -> Power - Output
