File: PCB_files/user_interface.kicad_sch (KiCad schematic)
At the start: 41 parts, among them J8 AFC07-S12FCA-00, Q7 AO3404A

Commit message: Update rotations
Parts:
- PZ1, Q7: FT Rotation Offset (none) -> 180
