File: PCB_files/Project Architecture.kicad_sch (KiCad schematic)
At the start: 8 parts

Commit message: Fix production files
Parts:
- renumbered MH2 to MH1, MH4 to MH2, MH5 to MH4, MH1 to MH5
Other:
- sheet MCU - Unit ports: added 5V_EN; removed 17V_EN
- sheet Power - Generation ports: added 5V_EN; removed 17V_EN
- title: Project Architecture -> Power - Output
