File: PCB_files/mcu_unit.kicad_sch (KiCad schematic)
At the start: 75 parts, among them J7 61300411121, U10 W25Q128JVPIQ, U9 RP2040, Y1 ABM8-272-T3

Commit message: Update 17V output to 5V output
Connections:
- net 17V_EN renamed 5V_EN
- net 17V_EN_R renamed 5V_EN_R

Commit message: Fix production files
Parts:
- C31: renamed from C44; MFR Part # (none) -> CL10B104KC8NNNC; Manufacturer Part Number CL10B104KC8NNNC -> (none)
- C32: renamed from C45; MFR Part # (none) -> 0402CG150J500NT; Manufacturer Part Number 0402CG150J500NT -> (none)
- C33: renamed from C46; MFR Part # (none) -> 0402CG150J500NT; Manufacturer Part Number 0402CG150J500NT -> (none)
- C34: renamed from C31; MFR Part # (none) -> CC0805KKX7R0BB105; Manufacturer Part Number CC0805KKX7R0BB105 -> (none)
- C35: renamed from C33; MFR Part # (none) -> CC0805KKX7R0BB105; Manufacturer Part Number CC0805KKX7R0BB105 -> (none)
- C36: MFR Part # (none) -> CC0805KKX7R0BB105; Manufacturer Part Number CC0805KKX7R0BB105 -> (none)
- C37: renamed from C32; MFR Part # (none) -> CC0805KKX7R0BB105; Manufacturer Part Number CC0805KKX7R0BB105 -> (none)
- C38: renamed from C34; MFR Part # (none) -> CL10B104KC8NNNC; Manufacturer Part Number CL10B104KC8NNNC -> (none)
- C39: renamed from C37; MFR Part # (none) -> CL10B104KC8NNNC; Manufacturer Part Number CL10B104KC8NNNC -> (none)
- C40: renamed from C35; MFR Part # (none) -> CL10B104KC8NNNC; Manufacturer Part Number CL10B104KC8NNNC -> (none)
- C41: renamed from C38; MFR Part # (none) -> CL10B104KC8NNNC; Manufacturer Part Number CL10B104KC8NNNC -> (none)
- C42: renamed from C39; MFR Part # (none) -> CL10B104KC8NNNC; Manufacturer Part Number CL10B104KC8NNNC -> (none)
- C43: renamed from C40; MFR Part # (none) -> CL10B104KC8NNNC; Manufacturer Part Number CL10B104KC8NNNC -> (none)
- C44: renamed from C41; MFR Part # (none) -> CL10B104KC8NNNC; Manufacturer Part Number CL10B104KC8NNNC -> (none)
- C45: renamed from C42; MFR Part # (none) -> CL10B104KC8NNNC; Manufacturer Part Number CL10B104KC8NNNC -> (none)
- C46: renamed from C43; MFR Part # (none) -> CL10B104KC8NNNC; Manufacturer Part Number CL10B104KC8NNNC -> (none)
- D10: renamed from D9; MFR Part # (none) -> APTD1608LQBC/D; Manufacturer Part Number APTD1608LQBC/D -> (none)
- D9: renamed from D10; MFR Part # (none) -> D3V3F4U6S-7; Manufacturer Part Number D3V3F4U6S-7 -> (none)
- J7: MFR Part # (none) -> 61300411121; Manufacturer Part Number 61300411121 -> (none)
- R35: renamed from R41; MFR Part # (none) -> 0402WGF1002TCE; Manufacturer Part Number 0402WGF1002TCE -> (none)
- R36: renamed from R63; MFR Part # (none) -> 0402WGF1001TCE; Manufacturer Part Number 0402WGF1001TCE -> (none)
- R37: renamed from R64; MFR Part # (none) -> RC0402FR-0727RL; Manufacturer Part Number RC0402FR-0727RL -> (none)
- R38: renamed from R66; MFR Part # (none) -> RC0402FR-0727RL; Manufacturer Part Number RC0402FR-0727RL -> (none)
- R39: renamed from R40; MFR Part # (none) -> RC0402FR-0727RL; Manufacturer Part Number RC0402FR-0727RL -> (none)
- R40: renamed from R42; MFR Part # (none) -> RC0402FR-0727RL; Manufacturer Part Number RC0402FR-0727RL -> (none)
- R41: renamed from R43; MFR Part # (none) -> RC0402FR-0727RL; Manufacturer Part Number RC0402FR-0727RL -> (none)
- R42: renamed from R44; MFR Part # (none) -> RC0402FR-0727RL; Manufacturer Part Number RC0402FR-0727RL -> (none)
- R43: renamed from R45; MFR Part # (none) -> RC0402FR-0727RL; Manufacturer Part Number RC0402FR-0727RL -> (none)
- R44: renamed from R46; MFR Part # (none) -> RC0402FR-0727RL; Manufacturer Part Number RC0402FR-0727RL -> (none)
- R45: renamed from R38; MFR Part # (none) -> RC0402FR-0727RL; Manufacturer Part Number RC0402FR-0727RL -> (none)
- R46: renamed from R39; MFR Part # (none) -> RC0402FR-0727RL; Manufacturer Part Number RC0402FR-0727RL -> (none)
- R47: renamed from R35; MFR Part # (none) -> 0402WGF1001TCE; Manufacturer Part Number 0402WGF1001TCE -> (none)
- R48: renamed from R47; MFR Part # (none) -> RC0402FR-0727RL; Manufacturer Part Number RC0402FR-0727RL -> (none)
- R49: renamed from R48; MFR Part # (none) -> RC0402FR-0727RL; Manufacturer Part Number RC0402FR-0727RL -> (none)
- R50: renamed from R49; MFR Part # (none) -> RC0402FR-0727RL; Manufacturer Part Number RC0402FR-0727RL -> (none)
- R51, R52, R56, R57, R58, R59, R60, R61: MFR Part # (none) -> RC0402FR-0727RL; Manufacturer Part Number RC0402FR-0727RL -> (none)
- R53, R54, R55: MFR Part # (none) -> 0402WGF1001TCE; Manufacturer Part Number 0402WGF1001TCE -> (none)
- R62: renamed from R65; MFR Part # (none) -> RC0402FR-0727RL; Manufacturer Part Number RC0402FR-0727RL -> (none)
- R63: renamed from R62; MFR Part # (none) -> RC0402FR-0727RL; Manufacturer Part Number RC0402FR-0727RL -> (none)
- R64: renamed from R67; MFR Part # (none) -> 0402WGF1001TCE; Manufacturer Part Number 0402WGF1001TCE -> (none)
- R65: renamed from R37; MFR Part # (none) -> RC0402FR-0727RL; Manufacturer Part Number RC0402FR-0727RL -> (none)
- R66: renamed from R36; MFR Part # (none) -> 0402WGF1002TCE; Manufacturer Part Number 0402WGF1002TCE -> (none)
- R67: renamed from R50; MFR Part # (none) -> 0402WGF3300TCE; Manufacturer Part Number 0402WGF3300TCE -> (none)
- S1, S2: MFR Part # (none) -> EVQ-PUC02K; Manufacturer Part Number EVQ-PUC02K -> (none)
- U10: renamed from U9; MFR Part # (none) -> SC0914(13); Manufacturer Part Number SC0914(13) -> (none)
- U9: renamed from U10; MFR Part # (none) -> W25Q128JVPIQ; Manufacturer Part Number W25Q128JVPIQ -> (none)
- Y1: MFR Part # (none) -> ABM8-272-T3; Manufacturer Part Number ABM8-272-T3 -> (none)
- renumbered TP47 to TP33, TP48 to TP34, TP49 to TP35, TP50 to TP36, TP33 to TP37, TP34 to TP38, TP35 to TP39, TP36 to TP40, TP37 to TP41, TP38 to TP42, TP39 to TP43, TP40 to TP44, TP41 to TP45, TP42 to TP46, TP43 to TP47, TP44 to TP48, TP45 to TP49, TP46 to TP50
Other:
- title: MCU - Unit -> Power - Output

Commit message: Update rotations
Parts:
- D9, Y1: FT Rotation Offset (none) -> 270
- S1, S2: FT Rotation Offset (none) -> 270; LCSC C79174 -> C79175; MFR Part # EVQ-PUC02K -> EVQPUL02K
- U9: FT Rotation Offset (none) -> 270; LCSC C190862 -> C2441427; MFR Part # W25Q128JVPIQ -> W25Q128JVPIM
