File: PCB_files/power_generation.kicad_sch (KiCad schematic)
At the start: 37 parts, among them U11 LMR16006XDDCR, U12 LMR16006XDDCR

Commit message: Update 17V output to 5V output
Parts:
- removed L2: 68uH 0.55A 0.91Ohm, Altium_port:SWPA4030S220MT, symbol Device:L
- removed R86: 10k 1%, Altium_port:resc_1005_04_n, symbol 0_passives:R_0402
- removed R89, R90: 4.7k 1%, Altium_port:resc_1005_04_m, symbol 0_passives:R_0402
- added L3: 33uH 1.3A 244mOhm, Inductor_SMD:L_APV_ANR5020, symbol Device:L_Small
- added R91, R92, R93: 10k 1%, Altium_port:resc_1005_04_n, symbol 0_passives:R_0402
- C67: value 10u X7R 63V -> 22u X7R 25V; LCSC C437568 -> C309062; Manufacturer Murata Electronics -> Samsung Electro-Mechanics; Manufacturer Part Number GRM32ER71J106KA12L -> CL32B226KAJNNNE
- R88: value 100k 1% -> 1k 1%; LCSC C25741 -> C11702; Manufacturer Part Number 0402WGF1003TCE -> 0402WGF1001TCE
Connections:
- net GND: now also R93.2
- net at R87.2: now also R91.1; no longer R88.1
- net +17V renamed +5V
- net +5V: now also R88.1, L3.2
- net 17V_CB renamed 5V_CB
- net 17V_EN renamed 5V_EN
- net 17V_FB renamed 5V_FB
- net 5V_FB: now also R91.2, R92.1; no longer R88.2
- net 17V_SW renamed 5V_SW
- net 5V_SW: now also L3.1
- net LED_17V_A renamed LED_5V_A
- net LED_5V_A: now also R88.2
- new net: R92.2, R93.1
Other:
- note added: "5V 600mA 700kHz Buck Regulator"
- note removed: "17V 600mA 700kHz Buck Regulator"
- moved on the sheet: C67, D14

Commit message: Fix production files
Parts:
- C55: renamed from C64; MFR Part # (none) -> CC0805KKX7R0BB105; Manufacturer Part Number CC0805KKX7R0BB105 -> (none)
- C56: MFR Part # (none) -> CC0805KKX7R0BB105; Manufacturer Part Number CC0805KKX7R0BB105 -> (none)
- C57: renamed from C65; MFR Part # (none) -> CC0805KKX7R0BB105; Manufacturer Part Number CC0805KKX7R0BB105 -> (none)
- C58: renamed from C57; MFR Part # (none) -> CC0805KKX7R0BB105; Manufacturer Part Number CC0805KKX7R0BB105 -> (none)
- C59: renamed from C66; MFR Part # (none) -> CC0805KKX7R0BB105; Manufacturer Part Number CC0805KKX7R0BB105 -> (none)
- C60: renamed from C58; MFR Part # (none) -> CC0805KKX7R0BB105; Manufacturer Part Number CC0805KKX7R0BB105 -> (none)
- C61: renamed from C62; MFR Part # (none) -> CC0805KKX7R0BB105; Manufacturer Part Number CC0805KKX7R0BB105 -> (none)
- C62: renamed from C63; MFR Part # (none) -> CL10B104KC8NNNC; Manufacturer Part Number CL10B104KC8NNNC -> (none)
- C63: renamed from C55; MFR Part # (none) -> CL10B104KC8NNNC; Manufacturer Part Number CL10B104KC8NNNC -> (none)
- C64: renamed from C67; MFR Part # (none) -> CL32B226KAJNNNE; Manufacturer Part Number CL32B226KAJNNNE -> (none)
- C65: renamed from C59; MFR Part # (none) -> GRM32ER71J106KA12L; Manufacturer Part Number GRM32ER71J106KA12L -> (none)
- C66: renamed from C60; MFR Part # (none) -> GRM32ER71J106KA12L; Manufacturer Part Number GRM32ER71J106KA12L -> (none)
- C67: renamed from C61; MFR Part # (none) -> GRM32ER71J106KA12L; Manufacturer Part Number GRM32ER71J106KA12L -> (none)
- D12: renamed from D13; MFR Part # (none) -> MBR1H100SFT3G; Manufacturer Part Number MBR1H100SFT3G -> (none)
- D13: renamed from D12; MFR Part # (none) -> MBR1H100SFT3G; Manufacturer Part Number MBR1H100SFT3G -> (none)
- D14: MFR Part # (none) -> APTD1608LQBC/D; Manufacturer Part Number APTD1608LQBC/D -> (none)
- L1: renamed from L3; MFR Part # (none) -> SMNR5040-330MT; Manufacturer Part Number SMNR5040-330MT -> (none)
- L2: renamed from L1; MFR Part # (none) -> SWPA4030S220MT; Manufacturer Part Number SWPA4030S220MT -> (none)
- R80: renamed from R85; MFR Part # (none) -> 0402WGF1003TCE; Manufacturer Part Number 0402WGF1003TCE -> (none)
- R81: MFR Part # (none) -> 0402WGF1003TCE; Manufacturer Part Number 0402WGF1003TCE -> (none)
- R82: MFR Part # (none) -> RC0402FR-0733KL; Manufacturer Part Number RC0402FR-0733KL -> (none)
- R83: renamed from R84; LCSC C25741 -> C25900; MFR Part # (none) -> 0402WGF4701TCE; Manufacturer Part Number 0402WGF1003TCE -> (none)
- R84: renamed from R87; MFR Part # (none) -> 0402WGF1003TCE; Manufacturer Part Number 0402WGF1003TCE -> (none)
- R85: renamed from R91; MFR Part # (none) -> 0402WGF1002TCE; Manufacturer Part Number 0402WGF1002TCE -> (none)
- R86: renamed from R92; MFR Part # (none) -> 0402WGF1002TCE; Manufacturer Part Number 0402WGF1002TCE -> (none)
- R87: renamed from R93; MFR Part # (none) -> 0402WGF1002TCE; Manufacturer Part Number 0402WGF1002TCE -> (none)
- R88: renamed from R80; MFR Part # (none) -> RC0402FR-0733KL; Manufacturer Part Number RC0402FR-0733KL -> (none)
- R89: renamed from R83; MFR Part # (none) -> 0402WGF1002TCE; Manufacturer Part Number 0402WGF1002TCE -> (none)
- R90: renamed from R88; MFR Part # (none) -> 0402WGF1001TCE; Manufacturer Part Number 0402WGF1001TCE -> (none)
- U11: renamed from U12; MFR Part # (none) -> LMR16006XDDCR; Manufacturer Part Number LMR16006XDDCR -> (none)
- U12: renamed from U11; MFR Part # (none) -> LMR16006XDDCR; Manufacturer Part Number LMR16006XDDCR -> (none)
Other:
- title: Power - Generation -> Power - Output

Commit message: Update rotations
Parts:
- U11, U12: FT Rotation Offset (none) -> 180
