File: PCB_files/power_pd_controller.kicad_sch (KiCad schematic)
At the start: 63 parts, among them J2 61300411121, Q3 SQJB90EP-T1_GE3, Q4 AO3404A, Q5 AO3404A, Q6 AO3404A, U2 LM2765, U3 TPS26750SRSMR, U4 LTC7004x, U5 74LVC1G08SE-7, U6 CAT24C512YI-GT3

Commit message: Fix production files
Parts:
- C10: renamed from C17; MFR Part # (none) -> CL10B104KC8NNNC; Manufacturer Part Number CL10B104KC8NNNC -> (none)
- C11: renamed from C19; MFR Part # (none) -> CL05B221KB5NNNC; Manufacturer Part Number CL05B221KB5NNNC -> (none)
- C12: renamed from C10; MFR Part # (none) -> GRM32ER71J106KA12L; Manufacturer Part Number GRM32ER71J106KA12L -> (none)
- C13: renamed from C20; MFR Part # (none) -> CL05B221KB5NNNC; Manufacturer Part Number CL05B221KB5NNNC -> (none)
- C14: renamed from C11; MFR Part # (none) -> GRM32ER71J106KA12L; Manufacturer Part Number GRM32ER71J106KA12L -> (none)
- C15: renamed from C12; MFR Part # (none) -> GRM32ER71J106KA12L; Manufacturer Part Number GRM32ER71J106KA12L -> (none)
- C16: renamed from C22; MFR Part # (none) -> CL10B104KC8NNNC; Manufacturer Part Number CL10B104KC8NNNC -> (none)
- C17: renamed from C13; MFR Part # (none) -> TCC0603X5R335M250CT; Manufacturer Part Number TCC0603X5R335M250CT -> (none)
- C18: renamed from C15; MFR Part # (none) -> TCC0603X5R335M250CT; Manufacturer Part Number TCC0603X5R335M250CT -> (none)
- C19: renamed from C14; MFR Part # (none) -> TCC0603X5R335M250CT; Manufacturer Part Number TCC0603X5R335M250CT -> (none)
- C20: renamed from C16; MFR Part # (none) -> CL10B104KC8NNNC; Manufacturer Part Number CL10B104KC8NNNC -> (none)
- C21: MFR Part # (none) -> CL10B104KC8NNNC; Manufacturer Part Number CL10B104KC8NNNC -> (none)
- C22: renamed from C18; MFR Part # (none) -> HHV0805R7225K101NSLJ; Manufacturer Part Number HHV0805R7225K101NSLJ -> (none)
- C9: MFR Part # (none) -> GRM32ER71J106KA12L; Manufacturer Part Number GRM32ER71J106KA12L -> (none)
- D5: renamed from D7; MFR Part # (none) -> D3V3F4U6S-7; Manufacturer Part Number D3V3F4U6S-7 -> (none)
- D6: renamed from D5; MFR Part # (none) -> B0520LW-7-F; Manufacturer Part Number B0520LW-7-F -> (none)
- D7: renamed from D6; MFR Part # (none) -> APTD1608LQBC/D; Manufacturer Part Number APTD1608LQBC/D -> (none)
- J2: MFR Part # (none) -> 61300411121; Manufacturer Part Number 61300411121 -> (none)
- Q3: renamed from Q4; MFR Part # (none) -> AO3404A; Manufacturer Part Number AO3404A -> (none)
- Q4: renamed from Q5; MFR Part # (none) -> AO3404A; Manufacturer Part Number AO3404A -> (none)
- Q5: renamed from Q3; MFR Part # (none) -> SQJB90EP-T1_GE3; Manufacturer Part Number SQJB90EP-T1_GE3 -> (none)
- Q6: MFR Part # (none) -> AO3404A; Manufacturer Part Number AO3404A -> (none)
- R10: renamed from R11; LCSC C25741 -> C25900; MFR Part # (none) -> 0402WGF4701TCE; Manufacturer Part Number 0402WGF1003TCE -> (none)
- R11: renamed from R12; LCSC C25741 -> C25900; MFR Part # (none) -> 0402WGF4701TCE; Manufacturer Part Number 0402WGF1003TCE -> (none)
- R12: renamed from R13; MFR Part # (none) -> 0402WGF1002TCE; Manufacturer Part Number 0402WGF1002TCE -> (none)
- R13: renamed from R21; MFR Part # (none) -> 0402WGF1003TCE; Manufacturer Part Number 0402WGF1003TCE -> (none)
- R14: renamed from R15; MFR Part # (none) -> 0402WGF1003TCE; Manufacturer Part Number 0402WGF1003TCE -> (none)
- R15: renamed from R16; MFR Part # (none) -> 0402WGF1003TCE; Manufacturer Part Number 0402WGF1003TCE -> (none)
- R16: renamed from R19; MFR Part # (none) -> 0402WGF1002TCE; Manufacturer Part Number 0402WGF1002TCE -> (none)
- R17: renamed from R18; LCSC C25741 -> C25900; MFR Part # (none) -> 0402WGF4701TCE; Manufacturer Part Number 0402WGF1003TCE -> (none)
- R18: renamed from R7; MFR Part # (none) -> RC0402FR-0727RL; Manufacturer Part Number RC0402FR-0727RL -> (none)
- R19: renamed from R14; MFR Part # (none) -> 0402WGF1003TCE; Manufacturer Part Number 0402WGF1003TCE -> (none)
- R20: renamed from R17; MFR Part # (none) -> 0402WGF1003TCE; Manufacturer Part Number 0402WGF1003TCE -> (none)
- R21: renamed from R20; MFR Part # (none) -> 0402WGF3300TCE; Manufacturer Part Number 0402WGF3300TCE -> (none)
- R7: renamed from R8; LCSC C25741 -> C25900; MFR Part # (none) -> 0402WGF4701TCE; Manufacturer Part Number 0402WGF1003TCE -> (none)
- R8: renamed from R9; LCSC C25741 -> C25900; MFR Part # (none) -> 0402WGF4701TCE; Manufacturer Part Number 0402WGF1003TCE -> (none)
- R9: renamed from R10; MFR Part # (none) -> 0402WGF1002TCE; Manufacturer Part Number 0402WGF1002TCE -> (none)
- U2: renamed from U3; MFR Part # (none) -> TPS26750SRSMR; Manufacturer Part Number TPS26750SRSMR -> (none)
- U3: renamed from U6; MFR Part # (none) -> CAT24C512YI-GT3; Manufacturer Part Number CAT24C512YI-GT3 -> (none)
- U4: renamed from U2; MFR Part # (none) -> LM2765M6X/NOPB; Manufacturer Part Number LM2765M6X/NOPB -> (none)
- U5: MFR Part # (none) -> 74LVC1G08SE-7; Manufacturer Part Number 74LVC1G08SE-7 -> (none)
- U6: renamed from U4; LCSC C690106 -> C690105; MFR Part # (none) -> LTC7004EMSE#PBF; Manufacturer Part Number LTC7004EMSE#TRPBF -> (none)
- renumbered JP3 to JP10, JP5 to JP3, JP7 to JP4, JP4 to JP5, JP8 to JP7, JP9 to JP8, JP10 to JP9, TP17 to TP15, TP19 to TP16, TP21 to TP17, TP23 to TP18, TP25 to TP19, TP15 to TP20, TP18 to TP21, TP20 to TP22, TP22 to TP23, TP26 to TP25, TP16 to TP26
Other:
- title: Power - PD Controller -> Power - Output

Commit message: Update rotations
Parts:
- D5, U2, U3, U5, U6: FT Rotation Offset (none) -> 270
- Q3, Q4, Q6, U4: FT Rotation Offset (none) -> 180
