File: PCB_files/power_sensing.kicad_sch (KiCad schematic)
At the start: 23 parts, among them U7 SN74LVC1G17DBVR, U8 INA228AIDGSR

Commit message: Fix production files
Parts:
- C23: renamed from C26; MFR Part # (none) -> CL10B104KC8NNNC; Manufacturer Part Number CL10B104KC8NNNC -> (none)
- C24: renamed from C27; MFR Part # (none) -> CL10B104KC8NNNC; Manufacturer Part Number CL10B104KC8NNNC -> (none)
- C25: renamed from C23; MFR Part # (none) -> CL10B104KC8NNNC; Manufacturer Part Number CL10B104KC8NNNC -> (none)
- C26: renamed from C24; MFR Part # (none) -> CL10B104KC8NNNC; Manufacturer Part Number CL10B104KC8NNNC -> (none)
- C27: renamed from C25; MFR Part # (none) -> CL10B104KC8NNNC; Manufacturer Part Number CL10B104KC8NNNC -> (none)
- R22: renamed from R27; MFR Part # (none) -> 0402WGF1003TCE; Manufacturer Part Number 0402WGF1003TCE -> (none)
- R23: renamed from R29; MFR Part # (none) -> 0402WGF1003TCE; Manufacturer Part Number 0402WGF1003TCE -> (none)
- R24: renamed from R31; MFR Part # (none) -> 0402WGF1002TCE; Manufacturer Part Number 0402WGF1002TCE -> (none)
- R25: renamed from R28; MFR Part # (none) -> 0402WGF1003TCE; Manufacturer Part Number 0402WGF1003TCE -> (none)
- R26: renamed from R30; LCSC C25741 -> C25900; MFR Part # (none) -> 0402WGF4701TCE; Manufacturer Part Number 0402WGF1003TCE -> (none)
- R27: renamed from R32; MFR Part # (none) -> SDNT1005X103F3950FTF; Manufacturer Part Number SDNT1005X103F3950FTF -> (none)
- R28: renamed from R23; MFR Part # (none) -> RC0402FR-0727RL; Manufacturer Part Number RC0402FR-0727RL -> (none)
- R29: renamed from R22; MFR Part # (none) -> HoLLR1206-1W-8mR-1%; Manufacturer Part Number HoLLR1206-1W-8mR-1% -> (none)
- R30: renamed from R24; MFR Part # (none) -> RC0402FR-0727RL; Manufacturer Part Number RC0402FR-0727RL -> (none)
- R31: renamed from R26; MFR Part # (none) -> RC0402FR-0727RL; Manufacturer Part Number RC0402FR-0727RL -> (none)
- R32: renamed from R25; LCSC C25741 -> C25900; MFR Part # (none) -> 0402WGF4701TCE; Manufacturer Part Number 0402WGF1003TCE -> (none)
- U7: renamed from U8; MFR Part # (none) -> INA228AIDGSR; Manufacturer Part Number INA228AIDGSR -> (none)
- U8: renamed from U7; MFR Part # (none) -> SN74LVC1G17DBVR; Manufacturer Part Number SN74LVC1G17DBVR -> (none)
Other:
- title: Power - Sensing -> Power - Output

Commit message: Update rotations
Parts:
- U7: FT Rotation Offset (none) -> 270; LCSC C2887910 -> C5214669
- U8: FT Rotation Offset (none) -> 180
