File: PCB_files/power_usb_c_input.kicad_sch (KiCad schematic)
At the start: 38 parts, among them J1 DX07S024JJ2R1300, Q1 AGM612AP, Q2 AO3404A, U1 TPD4S480RUKR

Commit message: Fix production files
Parts:
- C1: MFR Part # (none) -> CC0402KRX7R0BB103; Manufacturer Part Number CC0402KRX7R0BB103 -> (none)
- C2: renamed from C7; MFR Part # (none) -> CC0805KKX7R0BB105; Manufacturer Part Number CC0805KKX7R0BB105 -> (none)
- C3: renamed from C2; MFR Part # (none) -> CC0402KRX7R0BB103; Manufacturer Part Number CC0402KRX7R0BB103 -> (none)
- C4: renamed from C8; MFR Part # (none) -> CL10B104KC8NNNC; Manufacturer Part Number CL10B104KC8NNNC -> (none)
- C5: renamed from C3; MFR Part # (none) -> GCM32DC72A475KE02; Manufacturer Part Number GCM32DC72A475KE02 -> (none)
- C6: renamed from C4; MFR Part # (none) -> CL10B104KC8NNNC; Manufacturer Part Number CL10B104KC8NNNC -> (none)
- C7: renamed from C5; MFR Part # (none) -> CC0402KRX7R0BB103; Manufacturer Part Number CC0402KRX7R0BB103 -> (none)
- C8: renamed from C6; MFR Part # (none) -> CL10B104KC8NNNC; Manufacturer Part Number CL10B104KC8NNNC -> (none)
- D1: MFR Part # (none) -> SMAJ48A; Manufacturer Part Number SMAJ48A -> (none)
- D2, D3: MFR Part # (none) -> BZT52C18SQ; Manufacturer Part Number BZT52C18SQ -> (none)
- D4: MFR Part # (none) -> APTD1608LQBC/D; Manufacturer Part Number APTD1608LQBC/D -> (none)
- FB1: MFR Part # (none) -> BLM18SN220TH1D; Manufacturer Part Number BLM18SN220TH1D -> (none)
- J1: MFR Part # (none) -> DX07S024JJ2R1300; Manufacturer Part Number DX07S024JJ2R1300 -> (none)
- Q1: MFR Part # (none) -> AGM612AP; Manufacturer Part Number AGM612AP -> (none)
- Q2: MFR Part # (none) -> AO3404A; Manufacturer Part Number AO3404A -> (none)
- R1: renamed from R2; MFR Part # (none) -> RC0402FR-0733KL; Manufacturer Part Number RC0402FR-0733KL -> (none)
- R2: renamed from R6; MFR Part # (none) -> 0402WGF1002TCE; Manufacturer Part Number 0402WGF1002TCE -> (none)
- R3: renamed from R1; MFR Part # (none) -> 0402WGF1003TCE; Manufacturer Part Number 0402WGF1003TCE -> (none)
- R4: renamed from R3; MFR Part # (none) -> 0402WGF1003TCE; Manufacturer Part Number 0402WGF1003TCE -> (none)
- R5: renamed from R4; MFR Part # (none) -> RC0402FR-0733KL; Manufacturer Part Number RC0402FR-0733KL -> (none)
- R6: renamed from R5; MFR Part # (none) -> 0402WGF1001TCE; Manufacturer Part Number 0402WGF1001TCE -> (none)
- U1: MFR Part # (none) -> TPD4S480RUKR; Manufacturer Part Number TPD4S480RUKR -> (none)
- renumbered JP2 to JP1, JP1 to JP2, TP3 to TP1, TP1 to TP10, TP2 to TP11, TP4 to TP12, TP6 to TP13, TP5 to TP2, TP7 to TP3, TP8 to TP4, TP9 to TP5, TP10 to TP6, TP11 to TP7, TP12 to TP8, TP13 to TP9
Other:
- title: Power - USB-C Input -> Power - Output

Commit message: Update rotations
Parts:
- Q1, U1: FT Rotation Offset (none) -> 270
- Q2: FT Rotation Offset (none) -> 180
