File: hardware/Power - Sequencing.kicad_sch (KiCad schematic)
At the start: 0 parts

Commit message: Generate hardware documentation
Other:
- title: Power - Output -> Power - Sequencing
Changed lines of the file:
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@@
 	(paper "A3")
 	(title_block
-		(title "Power - Output")
+		(title "Power - Sequencing")
 		(date "2026-02-27")
 		(rev "${REVISION}")
