File: hardware/Project Architecture.kicad_sch (KiCad schematic)
At the start: 8 parts

Commit message: Generate hardware documentation
Other:
- sheet Power - Generation ports: added +5V; removed +17V
- sheet Power - Output ports: added +5V; removed +17V
- title: Power - Output -> Project Architecture
Changed lines of the file:
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@@
 	(paper "A3")
 	(title_block
-		(title "Power - Output")
+		(title "Project Architecture")
 		(date "2026-02-27")
 		(rev "${REVISION}")
@@
 			)
 		)
-		(pin "+17V" output
+		(pin "+5V" output
 			(at 196.85 181.61 0)
 			(effects
@@
 			)
 		)
-		(pin "+17V" input
+		(pin "+5V" input
 			(at 295.91 176.53 180)
 			(effects
