File: hardware/power_generation.kicad_sch (KiCad schematic)
At the start: 37 parts, among them U11 LMR16006XDDCR, U12 LMR16006XDDCR

Commit message: Generate hardware documentation
Other:
- title: Power - Output -> Power - Generation
Changed lines of the file:
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@@
 	(paper "A3")
 	(title_block
-		(title "Power - Output")
+		(title "Power - Generation")
 		(date "2026-02-27")
 		(rev "${REVISION}")
