File: hardware/power_pd_controller.kicad_sch (KiCad schematic)
At the start: 63 parts, among them J2 61300411121, Q3 AO3404A, Q4 AO3404A, Q5 SQJB90EP-T1_GE3, Q6 AO3404A, U2 TPS26750SRSMR, U3 CAT24C512YI-GT3, U4 LM2765, U5 74LVC1G08SE-7, U6 LTC7004x

Commit message: Generate hardware documentation
Other:
- title: Power - Output -> Power - PD Controller
Changed lines of the file:
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@@
 	(paper "A3")
 	(title_block
-		(title "Power - Output")
+		(title "Power - PD Controller")
 		(date "2026-02-27")
 		(rev "${REVISION}")
