File: hardware/power_sensing.kicad_sch (KiCad schematic)
At the start: 23 parts, among them U7 INA228AIDGSR, U8 SN74LVC1G17DBVR

Commit message: Generate hardware documentation
Other:
- title: Power - Output -> Power - Sensing
Changed lines of the file:
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@@
 	(paper "A3")
 	(title_block
-		(title "Power - Output")
+		(title "Power - Sensing")
 		(date "2026-02-27")
 		(rev "${REVISION}")
