File: hardware/user_interface.kicad_sch (KiCad schematic)
At the start: 41 parts, among them J8 AFC07-S12FCA-00, Q7 AO3404A

Commit message: Generate hardware documentation
Other:
- title: Power - Output -> User - Interface
Changed lines of the file:
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@@
 	(paper "A3")
 	(title_block
-		(title "Power - Output")
+		(title "User - Interface")
 		(date "2026-02-27")
 		(rev "${REVISION}")
